File: Avionics/ContraHopperFlightComputer/ContraHopperFlightComputer.kicad_pcb (KiCad board)
At the start: 2 copper layers, 1 part, among them U1 Teensy4.1

Commit message: flight_comptuer_draft_1
Parts:
- removed U1: Teensy4.1, UserKiCadFootprints:Teensy4.1
- added 5V_BUCK1: MINI-360, UserKiCadFootprints:MINI_360, F.Cu at (83.8, 150.9)
- added 8V_BUCK1: MINI-360, UserKiCadFootprints:MINI_360, F.Cu at (99.6, 150.9)
- added BARO1: GY-BMP280-3.3, UserKiCadFootprints:JST_XH_4pin, F.Cu at (49.8, 115.8)
- added BATT1: LIPO, UserKiCadFootprints:XT60_MOUNT, F.Cu at (101.6, 172.2)
- added BLUE1: LED, UserKiCadFootprints:LED, F.Cu at (77.7, 66.5)
- added GPS1: SparkFun_ZOE-M8Q, UserKiCadFootprints:SparkFun_ZOEM8Q, F.Cu at (65.5, 85.3)
- added IMU1: ISM330DHCX, UserKiCadFootprints:ISM330DHCX, F.Cu at (68.1, 119.4)
- added LIDAR1: TF_Mini_Plus, UserKiCadFootprints:JST_XH_4pin, F.Cu at (122.4, 113.8)
- added LM358: LM358, UserKiCadFootprints:LM358, F.Cu at (67.6, 146.8)
- added M1_POWER1: XING2/BL_HELI35A_POWER, UserKiCadFootprints:ESC_POWER, F.Cu at (85.3, 174.8)
- added M1_SIGNAL1: XING2/BL_HELI35A_SIGNAL, UserKiCadFootprints:JST_XH_2pin, F.Cu at (50.3, 148.3)
- added M2_POWER1: XING2/BL_HELI35A_POWER, UserKiCadFootprints:ESC_POWER, F.Cu at (68.1, 174.8)
- added M2_SIGNAL1: XING2/BL_HELI35A_SIGNAL, UserKiCadFootprints:JST_XH_2pin, F.Cu at (50.3, 158.0)
- added R1: R, UserKiCadFootprints:pinhole_resistor, F.Cu at (66.0, 159.5)
- added R2: R, UserKiCadFootprints:pinhole_resistor, F.Cu at (70.1, 159.5)
- added R3: R, UserKiCadFootprints:pinhole_resistor, F.Cu at (91.9, 77.7)
- added R4: R, UserKiCadFootprints:pinhole_resistor, F.Cu at (96.5, 77.7)
- added RADIO1: FS-IA6B, UserKiCadFootprints:FS-IA6B, F.Cu at (114.3, 92.6)
- added RED1: LED, UserKiCadFootprints:LED, F.Cu at (66.0, 66.5)
- added SV1: X06H_Servo, UserKiCadFootprints:JST_XH_3pin, F.Cu at (122.4, 158.0)
- added SV2: X06H_Servo, UserKiCadFootprints:JST_XH_3pin, F.Cu at (122.4, 147.3)
- added SV3: X06H_Servo, UserKiCadFootprints:JST_XH_3pin, F.Cu at (122.4, 136.7)
- added SV4: X06H_Servo, UserKiCadFootprints:JST_XH_3pin, F.Cu at (122.6, 126.0)
- added TEENSY1: Teensy4.1, UserKiCadFootprints:Teensy4.1, F.Cu at (94.0, 101.6)
Routing:
- net /BATT+: track 0.00 -> 109.1 mm
- net +5V: track 0.00 -> 105.6 mm, vias 0 -> 1
- net +3.3V: track 0.00 -> 84.1 mm
- net /SCL: track 0.00 -> 77.2 mm
- net /SDA: track 0.00 -> 73.4 mm
- net +8V: track 0.00 -> 57.2 mm
- net /M2_Signal: track 0.00 -> 55.3 mm, vias 0 -> 1
- net /BATT_LEVEL: track 0.00 -> 55.1 mm
- net /M1_Signal: track 0.00 -> 46.6 mm, vias 0 -> 1
- net /SV1_PWM: track 0.00 -> 46.0 mm
- net /SV2_PWM: track 0.00 -> 37.8 mm
- net /TX2: track 0.00 -> 31.4 mm
- net /SV3_PWM: track 0.00 -> 29.7 mm
- net Net-(R3-Pad1): track 0.00 -> 27.2 mm
- net /SV4_PWM: track 0.00 -> 26.3 mm
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- added copper zone on B.Cu, net GND
Other:
- board outline added: 77 x 116.3 mm
