File: Avionics/ContraHopperFlightComputer/ContraHopperFlightComputer.kicad_sch (KiCad schematic)
At the start: 1 part

Commit message: kicad fully integrated with git hub
Parts:
- removed U?: Teensy4.1, symbol teensy:Teensy4.1
- added U1: Teensy4.1, UserKiCadFootprints:Teensy4.1, symbol ContraHopperSymbols:Teensy4.1
Changed lines of the file:
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@@
 (kicad_sch (version 20211123) (generator eeschema)
   (paper "A4")
-  (symbol (lib_id "teensy:Teensy4.1") (at 147.32 86.36 0) (unit 1)
+  (symbol (lib_id "ContraHopperSymbols:Teensy4.1") (at 147.32 81.28 0) (unit 1)
     (in_bom yes) (on_board yes) (fields_autoplaced)
-    (property "Reference" "U?" (id 0) (at 147.32 20.32 0))
-    (property "Value" "Teensy4.1" (id 1) (at 147.32 22.86 0))
-    (property "Footprint" "" (id 2) (at 137.16 76.2 0)
+    (property "Reference" "U1" (id 0) (at 146.7247 27.94 0))
+    (property "Value" "Teensy4.1" (id 1) (at 146.7247 30.48 0))
+    (property "Footprint" "UserKiCadFootprints:Teensy4.1" (id 2) (at 147.32 83.82 0)
       (effects (font (size 1.27 1.27)) hide)
     )
-    (property "Datasheet" "" (id 3) (at 137.16 76.2 0)
+    (property "Datasheet" "" (id 3) (at 147.32 83.82 0)
       (effects (font (size 1.27 1.27)) hide)
     )
+    (pin "0")
+    (pin "1")
     (pin "10")
     (pin "11")
@@
     (pin "18")
     (pin "19")
+    (pin "2")
     (pin "20")
     (pin "21")
@@
     (pin "28")
     (pin "29")
+    (pin "3")
     (pin "30")
     (pin "31")
     (pin "32")
     (pin "33")
+    (pin "34")
     (pin "35")
     (pin "36")
@@
     (pin "38")
     (pin "39")
+    (pin "4")
     (pin "40")
     (pin "41")
-    (pin "42")
     (pin "43")
     (pin "44")
@@
     (pin "47")
     (pin "48")
-    (pin "49")
     (pin "5")
-    (pin "50")
-    (pin "51")
-    (pin "52")
-    (pin "53")
-    (pin "54")
-    (pin "55")
-    (pin "56")
-    (pin "57")
-    (pin "58")
-    (pin "59")
     (pin "6")
-    (pin "60")
-    (pin "61")
-    (pin "62")
-    (pin "63")
-    (pin "64")
-    (pin "65")
-    (pin "66")
-    (pin "67")
     (pin "7")
     (pin "8")
     (pin "9")
-    (pin "1")
-    (pin "2")
-    (pin "3")
-    (pin "34")
-    (pin "4")
   )
   (sheet_instances
@@
   )
   (symbol_instances
-    (path "/d8e83bb6-4f27-4786-9375-f9b709397f23"
-      (reference "U?") (unit 1) (value "Teensy4.1") (footprint "")
+    (path "/aff048f3-aa9a-4e9f-8543-32a07df71fe3"
+      (reference "U1") (unit 1) (value "Teensy4.1") (footprint "UserKiCadFootprints:Teensy4.1")
     )
   )

Commit message: flight_comptuer_draft_1
Parts:
- added 5V_BUCK1, 8V_BUCK1: MINI-360, UserKiCadFootprints:MINI_360, symbol ContraHopperSymbols:MINI-360
- added BARO1: GY-BMP280-3.3, UserKiCadFootprints:JST_XH_4pin, symbol ContraHopperSymbols:GY-BMP280-3.3
- added BATT1: LIPO, UserKiCadFootprints:XT60_MOUNT, symbol ContraHopperSymbols:LIPO
- added BLUE1, RED1: LED, UserKiCadFootprints:LED, symbol Device:LED
- added GPS1: SparkFun_ZOE-M8Q, UserKiCadFootprints:SparkFun_ZOEM8Q, symbol ContraHopperSymbols:SparkFun_ZOE-M8Q
- added IMU1: ISM330DHCX, UserKiCadFootprints:ISM330DHCX, symbol ContraHopperSymbols:ISM330DHCX
- added LIDAR1: TF_Mini_Plus, UserKiCadFootprints:JST_XH_4pin, symbol ContraHopperSymbols:TF_Mini_Plus
- added LM358: LM358, UserKiCadFootprints:LM358, symbol ContraHopperSymbols:LM358
- added M1_POWER1, M2_POWER1: XING2/BL_HELI35A_POWER, UserKiCadFootprints:ESC_POWER, symbol ContraHopperSymbols:XING2/BL_HELI35A_POWER
- added M1_SIGNAL1, M2_SIGNAL1: XING2/BL_HELI35A_SIGNAL, UserKiCadFootprints:JST_XH_2pin, symbol ContraHopperSymbols:XING2/BL_HELI35A_SIGNAL
- added R1, R2, R3, R4: R, UserKiCadFootprints:pinhole_resistor, symbol Device:R
- added RADIO1: FS-IA6B, UserKiCadFootprints:FS-IA6B, symbol ContraHopperSymbols:FS-IA6B
- added SV1, SV2, SV3, SV4: X06H_Servo, UserKiCadFootprints:JST_XH_3pin, symbol ContraHopperSymbols:X06H_Servo
- renumbered U1 to TEENSY1
Connections:
- net CH4: now reaches TEENSY1.10
- net CH4: now also RADIO1.4 (CH4)
- net CH3: now reaches TEENSY1.11
- net CH3: now also RADIO1.3 (CH3)
- net CH2: now reaches TEENSY1.12
- net CH2: now also RADIO1.2 (CH2)
- net SDA: now reaches TEENSY1.18 (SDA)
- net SDA: now also BARO1.4 (SDA), GPS1.8 (SDA), IMU1.5 (SDA)
- net SCL: now reaches TEENSY1.19 (SCL)
- net SCL: now also BARO1.3 (SCL), GPS1.7 (SCL), IMU1.4 (SCL)
- net SV1_PWM: now reaches TEENSY1.2
- net SV1_PWM: now also SV1.1 (PWM)
- net BATT_LEVEL: now reaches TEENSY1.21 (A7)
- net BATT_LEVEL: now also LM358.2 (-), LM358.3
- net M2_Signal: now reaches TEENSY1.22 (A8)
- net M2_Signal: now also M2_SIGNAL1.1 (S+)
- net M1_Signal: now reaches TEENSY1.23 (A9)
- net M1_Signal: now also M1_SIGNAL1.1 (S+)
- net CH1: now reaches TEENSY1.24 (A10(SCL2))
- net CH1: now also RADIO1.1 (CH1)
- net BLUE_LED: now reaches TEENSY1.26 (A12)
- net BLUE_LED: now also R3.2
- net RED_LED: now reaches TEENSY1.27 (A13)
- net RED_LED: now also R4.2
- net SV2_PWM: now reaches TEENSY1.3
- net SV2_PWM: now also SV2.1 (PWM)
- net SV3_PWM: now reaches TEENSY1.4
- net SV3_PWM: now also SV3.1 (PWM)
- net GND: now reaches TEENSY1.43 (GND)
- net GND: now also TEENSY1.46 (GND), TEENSY1.48 (GND), 5V_BUCK1.2 (VIN-), 5V_BUCK1.3 (VOUT-), 8V_BUCK1.2 (VIN-), 8V_BUCK1.3 (VOUT-), BARO1.2 (GND), BATT1.2 (BATT-), BLUE1.2 (A), GPS1.6 (GND), IMU1.14 (GND), IMU1.3 (GND), LIDAR1.4 (GND), LM358.5 (V-), M1_POWER1.2 (BATT-), M1_SIGNAL1.2 (S-), M2_POWER1.2 (BATT-), M2_SIGNAL1.2 (S-), R2.2, RADIO1.9 (GND), RED1.2 (A), SV1.3 (GND), SV2.3 (GND), SV3.3 (GND), SV4.3 (GND)
- net +5V: now reaches TEENSY1.45 (Vin)
- net +5V: now also 5V_BUCK1.4 (VOUT+), IMU1.1 (VIN), LIDAR1.1 (+5V), RADIO1.8 (VCC)
- net +3.3V: now reaches TEENSY1.47 (3.3v(250ma))
- net +3.3V: now also BARO1.1 (3.3V), GPS1.4 (3V3)
- net SV4_PWM: now reaches TEENSY1.5
- net SV4_PWM: now also SV4.1 (PWM)
- net CH6: now reaches TEENSY1.6
- net CH6: now also RADIO1.6 (CH6)
- net RX2: now reaches TEENSY1.7 (RX2)
- net RX2: now also LIDAR1.3 (TXD)
- net TX2: now reaches TEENSY1.8 (TX2)
- net TX2: now also LIDAR1.2 (RXD)
- net CH5: now reaches TEENSY1.9
- net CH5: now also RADIO1.5 (CH5)
- new net: LM358.1 (+), R1.2, R2.1
- new net: BLUE1.1 (K), R4.1
- new net: R3.1, RED1.1 (K)
- new net +8V: 8V_BUCK1.4 (VOUT+), SV1.2 (5V-8V), SV2.2 (5V-8V), SV3.2 (5V-8V), SV4.2 (5V-8V)
- new net BATT+: 5V_BUCK1.1 (VIN+), 8V_BUCK1.1 (VIN+), BATT1.1 (BATT+), LM358.4 (V+), M1_POWER1.1 (BATT+), M2_POWER1.1 (BATT+), R1.1
Other:
- note added: "MCU"
- note added: "MISC"
- note added: "MOTORS"
- note added: "Power"
- note added: "RADIO"
- note added: "SENSORS"
- note added: "SERVOS"
- moved on the sheet: TEENSY1
