File: Avionics/FlightBread/FlightBread.kicad_pcb (KiCad board)
At the start: 2 copper layers, 77 x 116.3 mm, 24 parts, among them M1_POWER1 XING2/BL_HELI35A_POWER, M1_SIGNAL1 XING2/BL_HELI35A_SIGNAL, M2_POWER1 XING2/BL_HELI35A_POWER, M2_SIGNAL1 XING2/BL_HELI35A_SIGNAL

Commit message: flight bread and more
Parts:
- R1: value R -> 6k
- R2: value R -> 2k
- moved M2_POWER1 3.45 mm to (70.9, 172.7)
- moved M1_POWER1 2.03 mm to (85.3, 172.7)
- moved BATT1 2.03 mm to (101.6, 170.2)
- moved BARO1 1.52 mm to (51.3, 115.8)
- moved M1_SIGNAL1 1.02 mm to (51.3, 148.3)
- moved M2_SIGNAL1 1.02 mm to (51.3, 158.0)
- moved SV4 0.91 mm to (121.7, 126.0)
- moved LIDAR1 0.76 mm to (121.7, 113.8)
- moved RADIO1 0.76 mm to (113.5, 92.6)
- moved SV1 0.76 mm to (121.7, 158.0)
- moved SV2 0.76 mm to (121.7, 147.3)
- moved SV3 0.76 mm to (121.7, 136.7)
Routing:
- net /BATT+: track 109.1 -> 100.1 mm
- net +8V: track 57.2 -> 54.3 mm
- net /SDA: track 73.4 -> 71.2 mm
- net /M1_Signal: track 46.6 -> 45.5 mm
- net /SV4_PWM: track 26.3 -> 25.4 mm
- net GND: track 4.91 -> 3.99 mm, vias 4 -> 2
- net /SCL: track 77.2 -> 76.4 mm
- net /RX2: track 21.7 -> 20.9 mm
- net +3.3V: track 84.1 -> 84.8 mm
- net /TX2: track 31.4 -> 30.8 mm
- net /CH2: track 14.5 -> 15.0 mm
- net /CH5: track 14.5 -> 15.0 mm
- net /CH4: track 14.5 -> 15.0 mm
- net /CH3: track 14.5 -> 15.0 mm
Other:
- board size 77 x 116.3 mm -> 77 x 116 mm
