File: Avionics/FlightBread/FlightBread.kicad_sch (KiCad schematic)
At the start: 24 parts, among them M1_POWER1 XING2/BL_HELI35A_POWER, M1_SIGNAL1 XING2/BL_HELI35A_SIGNAL, M2_POWER1 XING2/BL_HELI35A_POWER, M2_SIGNAL1 XING2/BL_HELI35A_SIGNAL

Commit message: folder_structure_update
Parts:
- renumbered RED1 to BLUE1, BLUE1 to RED1
Changed lines of the file:
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@@
   (symbol (lib_id "Device:LED") (at 209.55 50.8 0) (unit 1)
     (in_bom yes) (on_board yes)
-    (property "Reference" "BLUE1" (id 0) (at 208.28 57.15 0))
+    (property "Reference" "RED1" (id 0) (at 208.28 57.15 0))
     (property "Value" "LED" (id 1) (at 208.28 54.61 0))
     (property "Footprint" "UserKiCadFootprints:LED" (id 2) (at 209.55 50.8 0)
@@
   (symbol (lib_id "Device:LED") (at 209.55 39.37 0) (unit 1)
     (in_bom yes) (on_board yes) (fields_autoplaced)
-    (property "Reference" "RED1" (id 0) (at 207.9625 33.02 0))
+    (property "Reference" "BLUE1" (id 0) (at 207.9625 33.02 0))
     (property "Value" "LED" (id 1) (at 207.9625 35.56 0))
     (property "Footprint" "UserKiCadFootprints:LED" (id 2) (at 209.55 39.37 0)
@@
       (reference "BATT1") (unit 1) (value "LIPO") (footprint "UserKiCadFootprints:XT60_MOUNT")
     )
-    (path "/ee74ff6d-b41f-4c74-a993-13dd5c25e99b"
+    (path "/fe1c6224-af8a-4cd4-aba7-4fdcb9e56bf0"
       (reference "BLUE1") (unit 1) (value "LED") (footprint "UserKiCadFootprints:LED")
     )
@@
       (reference "RADIO1") (unit 1) (value "FS-IA6B") (footprint "UserKiCadFootprints:FS-IA6B")
     )
-    (path "/fe1c6224-af8a-4cd4-aba7-4fdcb9e56bf0"
+    (path "/ee74ff6d-b41f-4c74-a993-13dd5c25e99b"
       (reference "RED1") (unit 1) (value "LED") (footprint "UserKiCadFootprints:LED")
     )
